Commit message: Add files via upload

File: mr_robot_description/urdf/mr_robot.xacro (robot description, xacro)
@@ -3,11 +3,10 @@
 <xacro:include filename="$(find mr_robot_description)/urdf/materials.xacro" />
 <xacro:include filename="$(find mr_robot_description)/urdf/mr_robot.trans" />
-<xacro:include filename="$(find mr_robot_description)/gazebo/mr_robot.gazebo" />
-<xacro:include filename="$(find mr_robot_description)/gazebo/mr_robot_plugins.gazebo" />
+<xacro:include filename="$(find mr_robot_description)/urdf/mr_robot.gazebo" />
 <link name="base_link">
   <inertial>
-    <origin rpy="0 0 0" xyz="-0.003126400273591084 -0.020689296000987453 0.046454333142005186"/>
-    <mass value="0.7292137164141753"/>
-    <inertia ixx="0.007525" ixy="-2e-06" ixz="3e-06" iyy="0.007431" iyz="0.000242" izz="0.01454"/>
+    <origin rpy="0 0 0" xyz="-0.0183828854411911 -9.351398117062208e-17 0.047762106966911216"/>
+    <mass value="0.6932522980076122"/>
+    <inertia ixx="0.007399" ixy="-0.0" ixz="0.000221" iyy="0.006915" iyz="-0.0" izz="0.013959"/>
   </inertial>
   <visual>
@@ -25,121 +24,121 @@
   </collision>
 </link>
-<link name="R_motor_clamp__1__1">
-  <inertial>
-    <origin rpy="0 0 0" xyz="0.0697931404049471 0.00337936338359856 0.01067445022870011"/>
+<link name="L_motor_1">
+  <inertial>
+    <origin rpy="0 0 0" xyz="0.01549999996857043 -0.027245319885060224 -0.00017182896795726876"/>
+    <mass value="0.41014753708080764"/>
+    <inertia ixx="0.000183" ixy="0.0" ixz="0.0" iyy="5.4e-05" iyz="3e-06" izz="0.000183"/>
+  </inertial>
+  <visual>
+    <origin rpy="0 0 0" xyz="0.01275 -0.071 -0.0602"/>
+    <geometry>
+      <mesh filename="package://mr_robot_description/meshes/L_motor_1.stl" scale="0.001 0.001 0.001"/>
+    </geometry>
+    <material name="silver"/>
+  </visual>
+  <collision>
+    <origin rpy="0 0 0" xyz="0.01275 -0.071 -0.0602"/>
+    <geometry>
+      <mesh filename="package://mr_robot_description/meshes/L_motor_1.stl" scale="0.001 0.001 0.001"/>
+    </geometry>
+  </collision>
+</link>
+<link name="R_motor_1">
+  <inertial>
+    <origin rpy="0 0 0" xyz="-0.015499999968570767 0.027245319885060487 -0.00017182896795692876"/>
+    <mass value="0.41014753708080764"/>
+    <inertia ixx="0.000183" ixy="0.0" ixz="-0.0" iyy="5.4e-05" iyz="-3e-06" izz="0.000183"/>
+  </inertial>
+  <visual>
+    <origin rpy="0 0 0" xyz="-0.01775 0.071 -0.0602"/>
+    <geometry>
+      <mesh filename="package://mr_robot_description/meshes/R_motor_1.stl" scale="0.001 0.001 0.001"/>
+    </geometry>
+    <material name="silver"/>
+  </visual>
+  <collision>
+    <origin rpy="0 0 0" xyz="-0.01775 0.071 -0.0602"/>
+    <geometry>
+      <mesh filename="package://mr_robot_description/meshes/R_motor_1.stl" scale="0.001 0.001 0.001"/>
+    </geometry>
+  </collision>
+</link>
+<link name="R_wheel_1">
+  <inertial>
+    <origin rpy="0 0 0" xyz="1.7455221296147627e-14 -0.006133491954579948 -9.020562075079397e-15"/>
+    <mass value="0.33673316347081705"/>
+    <inertia ixx="0.000211" ixy="-0.0" ixz="-0.0" iyy="0.000351" iyz="0.0" izz="0.000211"/>
+  </inertial>
+  <visual>
+    <origin rpy="0 0 0" xyz="-0.00225 0.0997 -0.0534"/>
+    <geometry>
+      <mesh filename="package://mr_robot_description/meshes/R_wheel_1.stl" scale="0.001 0.001 0.001"/>
+    </geometry>
+    <material name="silver"/>
+  </visual>
+  <collision>
+    <origin rpy="0 0 0" xyz="-0.00225 0.0997 -0.0534"/>
+    <geometry>
+      <mesh filename="package://mr_robot_description/meshes/R_wheel_1.stl" scale="0.001 0.001 0.001"/>
+    </geometry>
+  </collision>
+</link>
+<link name="L_wheel_1">
+  <inertial>
+    <origin rpy="0 0 0" xyz="-1.705927066275592e-14 0.006133491954580114 -1.004057947895376e-14"/>
+    <mass value="0.33673316347081705"/>
+    <inertia ixx="0.000211" ixy="-0.0" ixz="0.0" iyy="0.000351" iyz="-0.0" izz="0.000211"/>
+  </inertial>
+  <visual>
+    <origin rpy="0 0 0" xyz="-0.00275 -0.0997 -0.0534"/>
+    <geometry>
+      <mesh filename="package://mr_robot_description/meshes/L_wheel_1.stl" scale="0.001 0.001 0.001"/>
+    </geometry>
+    <material name="silver"/>
+  </visual>
+  <collision>
+    <origin rpy="0 0 0" xyz="-0.00275 -0.0997 -0.0534"/>
+    <geometry>
+      <mesh filename="package://mr_robot_description/meshes/L_wheel_1.stl" scale="0.001 0.001 0.001"/>
+    </geometry>
+  </collision>
+</link>
+<link name="L_motor_clamp_1">
+  <inertial>
+    <origin rpy="0 0 0" xyz="-8.07643882327902e-15 0.0665047179820893 0.0107653911894319"/>
     <mass value="0.019214264346508234"/>
-    <inertia ixx="7e-06" ixy="0.0" ixz="-1e-06" iyy="4e-06" iyz="0.0" izz="4e-06"/>
-  </inertial>
-  <visual>
-    <origin rpy="0 0 0" xyz="0.006577 0.004259 -0.040182"/>
-    <geometry>
-      <mesh filename="package://mr_robot_description/meshes/R_motor_clamp__1__1.stl" scale="0.001 0.001 0.001"/>
-    </geometry>
-    <material name="silver"/>
-  </visual>
-  <collision>
-    <origin rpy="0 0 0" xyz="0.006577 0.004259 -0.040182"/>
-    <geometry>
-      <mesh filename="package://mr_robot_description/meshes/R_motor_clamp__1__1.stl" scale="0.001 0.001 0.001"/>
-    </geometry>
-  </collision>
-</link>
-<link name="L_motor_clamp_1">
-  <inertial>
-    <origin rpy="0 0 0" xyz="-0.0632162955592317 0.0033793633835824217 0.010674450228699485"/>
+    <inertia ixx="4e-06" ixy="-0.0" ixz="-0.0" iyy="7e-06" iyz="-1e-06" izz="4e-06"/>
+  </inertial>
+  <visual>
+    <origin rpy="0 0 0" xyz="-0.0025 0.0 -0.04"/>
+    <geometry>
+      <mesh filename="package://mr_robot_description/meshes/L_motor_clamp_1.stl" scale="0.001 0.001 0.001"/>
+    </geometry>
+    <material name="silver"/>
+  </visual>
+  <collision>
+    <origin rpy="0 0 0" xyz="-0.0025 0.0 -0.04"/>
+    <geometry>
+      <mesh filename="package://mr_robot_description/meshes/L_motor_clamp_1.stl" scale="0.001 0.001 0.001"/>
+    </geometry>
+  </collision>
+</link>
+<link name="R_motor_clamp_1">
+  <inertial>
+    <origin rpy="0 0 0" xyz="8.05995895025724e-15 -0.06650471798208926 0.010765391189432517"/>
     <mass value="0.019214264346508234"/>
-    <inertia ixx="7e-06" ixy="0.0" ixz="1e-06" iyy="4e-06" iyz="-0.0" izz="4e-06"/>
-  </inertial>
-  <visual>
-    <origin rpy="0 0 0" xyz="0.006577 0.004259 -0.040182"/>
-    <geometry>
-      <mesh filename="package://mr_robot_description/meshes/L_motor_clamp_1.stl" scale="0.001 0.001 0.001"/>
-    </geometry>
-    <material name="silver"/>
-  </visual>
-  <collision>
-    <origin rpy="0 0 0" xyz="0.006577 0.004259 -0.040182"/>
-    <geometry>
-      <mesh filename="package://mr_robot_description/meshes/L_motor_clamp_1.stl" scale="0.001 0.001 0.001"/>
-    </geometry>
-  </collision>
-</link>
-<link name="L_motor_1">
-  <inertial>
-    <origin rpy="0 0 0" xyz="0.027245742307917993 0.015500363352160937 -0.0001717699286896482"/>
-    <mass value="0.41014753708080764"/>
-    <inertia ixx="5.4e-05" ixy="-0.0" ixz="-3e-06" iyy="0.000183" iyz="0.0" izz="0.000183"/>
-  </inertial>
-  <visual>
-    <origin rpy="0 0 0" xyz="0.074289 0.01613 -0.060291"/>
-    <geometry>
-      <mesh filename="package://mr_robot_description/meshes/L_motor_1.stl" scale="0.001 0.001 0.001"/>
-    </geometry>
-    <material name="silver"/>
-  </visual>
-  <collision>
-    <origin rpy="0 0 0" xyz="0.074289 0.01613 -0.060291"/>
-    <geometry>
-      <mesh filename="package://mr_robot_description/meshes/L_motor_1.stl" scale="0.001 0.001 0.001"/>
-    </geometry>
-  </collision>
-</link>
-<link name="R_motor_1">
-  <inertial>
-    <origin rpy="0 0 0" xyz="-0.027244897462202544 -0.015499636584980275 -0.00017176992868937757"/>
-    <mass value="0.41014753708080764"/>
-    <inertia ixx="5.4e-05" ixy="-0.0" ixz="3e-06" iyy="0.000183" iyz="-0.0" izz="0.000183"/>
-  </inertial>
-  <visual>
-    <origin rpy="0 0 0" xyz="-0.067711 -0.01437 -0.060291"/>
-    <geometry>
-      <mesh filename="package://mr_robot_description/meshes/R_motor_1.stl" scale="0.001 0.001 0.001"/>
-    </geometry>
-    <material name="silver"/>
-  </visual>
-  <collision>
-    <origin rpy="0 0 0" xyz="-0.067711 -0.01437 -0.060291"/>
-    <geometry>
-      <mesh filename="package://mr_robot_description/meshes/R_motor_1.stl" scale="0.001 0.001 0.001"/>
-    </geometry>
-  </collision>
-</link>
-<link name="R_wheel_1">
-  <inertial>
-    <origin rpy="0 0 0" xyz="0.006133914377437905 3.633836079468093e-07 5.9039258544502093e-08"/>
-    <mass value="0.33673316347081705"/>
-    <inertia ixx="0.000351" ixy="0.0" ixz="-0.0" iyy="0.000211" iyz="-0.0" izz="0.000211"/>
-  </inertial>
-  <visual>
-    <origin rpy="0 0 0" xyz="-0.096411 0.00113 -0.053491"/>
-    <geometry>
-      <mesh filename="package://mr_robot_description/meshes/R_wheel_1.stl" scale="0.001 0.001 0.001"/>
-    </geometry>
-    <material name="silver"/>
-  </visual>
-  <collision>
-    <origin rpy="0 0 0" xyz="-0.096411 0.00113 -0.053491"/>
-    <geometry>
-      <mesh filename="package://mr_robot_description/meshes/R_wheel_1.stl" scale="0.001 0.001 0.001"/>
-    </geometry>
-  </collision>
-</link>
-<link name="L_wheel_1">
-  <inertial>
-    <origin rpy="0 0 0" xyz="-0.006133069531722379 3.633835734508572e-07 5.903925759387363e-08"/>
-    <mass value="0.33673316347081705"/>
-    <inertia ixx="0.000351" ixy="0.0" ixz="0.0" iyy="0.000211" iyz="0.0" izz="0.000211"/>
-  </inertial>
-  <visual>
-    <origin rpy="0 0 0" xyz="0.102989 0.00063 -0.053491"/>
-    <geometry>
-      <mesh filename="package://mr_robot_description/meshes/L_wheel_1.stl" scale="0.001 0.001 0.001"/>
-    </geometry>
-    <material name="silver"/>
-  </visual>
-  <collision>
-    <origin rpy="0 0 0" xyz="0.102989 0.00063 -0.053491"/>
-    <geometry>
-      <mesh filename="package://mr_robot_description/meshes/L_wheel_1.stl" scale="0.001 0.001 0.001"/>
+    <inertia ixx="4e-06" ixy="-0.0" ixz="0.0" iyy="7e-06" iyz="1e-06" izz="4e-06"/>
+  </inertial>
+  <visual>
+    <origin rpy="0 0 0" xyz="-0.0025 0.0 -0.04"/>
+    <geometry>
+      <mesh filename="package://mr_robot_description/meshes/R_motor_clamp_1.stl" scale="0.001 0.001 0.001"/>
+    </geometry>
+    <material name="silver"/>
+  </visual>
+  <collision>
+    <origin rpy="0 0 0" xyz="-0.0025 0.0 -0.04"/>
+    <geometry>
+      <mesh filename="package://mr_robot_description/meshes/R_motor_clamp_1.stl" scale="0.001 0.001 0.001"/>
     </geometry>
   </collision>
@@ -147,10 +146,10 @@
 <link name="motor_driver_1">
   <inertial>
-    <origin rpy="0 0 0" xyz="0.0024521933363072677 -0.04491646621231004 0.007099979095499857"/>
+    <origin rpy="0 0 0" xyz="-0.043295829595900504 0.0008362290865504151 0.00719092005623221"/>
     <mass value="0.016082198290596435"/>
-    <inertia ixx="3e-06" ixy="-0.0" ixz="-0.0" iyy="2e-06" iyz="-1e-06" izz="4e-06"/>
-  </inertial>
-  <visual>
-    <origin rpy="0 0 0" xyz="0.006577 0.004259 -0.040182"/>
+    <inertia ixx="2e-06" ixy="0.0" ixz="-1e-06" iyy="3e-06" iyz="0.0" izz="4e-06"/>
+  </inertial>
+  <visual>
+    <origin rpy="0 0 0" xyz="-0.0025 0.0 -0.04"/>
     <geometry>
       <mesh filename="package://mr_robot_description/meshes/motor_driver_1.stl" scale="0.001 0.001 0.001"/>
@@ -159,5 +158,5 @@
   </visual>
   <collision>
-    <origin rpy="0 0 0" xyz="0.006577 0.004259 -0.040182"/>
+    <origin rpy="0 0 0" xyz="-0.0025 0.0 -0.04"/>
     <geometry>
       <mesh filename="package://mr_robot_description/meshes/motor_driver_1.stl" scale="0.001 0.001 0.001"/>
@@ -167,10 +166,10 @@
 <link name="battery_1">
   <inertial>
-    <origin rpy="0 0 0" xyz="0.0023322069987047273 0.04337936338359042 0.016909059039267572"/>
+    <origin rpy="0 0 0" xyz="0.03999999999999985 0.0009562154241530774 0.017000000000000022"/>
     <mass value="0.49636285277615166"/>
-    <inertia ixx="6.9e-05" ixy="0.0" ixz="0.0" iyy="0.000509" iyz="0.0" izz="0.000483"/>
-  </inertial>
-  <visual>
-    <origin rpy="0 0 0" xyz="0.006577 0.004259 -0.040182"/>
+    <inertia ixx="0.000509" ixy="-0.0" ixz="0.0" iyy="6.9e-05" iyz="-0.0" izz="0.000483"/>
+  </inertial>
+  <visual>
+    <origin rpy="0 0 0" xyz="-0.0025 0.0 -0.04"/>
     <geometry>
       <mesh filename="package://mr_robot_description/meshes/battery_1.stl" scale="0.001 0.001 0.001"/>
@@ -179,5 +178,5 @@
   </visual>
   <collision>
-    <origin rpy="0 0 0" xyz="0.006577 0.004259 -0.040182"/>
+    <origin rpy="0 0 0" xyz="-0.0025 0.0 -0.04"/>
     <geometry>
       <mesh filename="package://mr_robot_description/meshes/battery_1.stl" scale="0.001 0.001 0.001"/>
@@ -187,10 +186,10 @@
 <link name="cover_1">
   <inertial>
-    <origin rpy="0 0 0" xyz="0.003427499441474675 0.14726742892395694 0.002403319815094937"/>
+    <origin rpy="0 0 0" xyz="0.143794391136608 -0.00013907701861727573 0.0024942607758274143"/>
     <mass value="3.0449746602441645"/>
-    <inertia ixx="0.025731" ixy="1e-05" ixz="-0.0" iyy="0.021423" iyz="3e-06" izz="0.047142"/>
-  </inertial>
-  <visual>
-    <origin rpy="0 0 0" xyz="0.006577 0.151759 -0.090182"/>
+    <inertia ixx="0.021423" ixy="-1e-05" ixz="3e-06" iyy="0.025731" iyz="0.0" izz="0.047142"/>
+  </inertial>
+  <visual>
+    <origin rpy="0 0 0" xyz="0.145 -0.0 -0.09"/>
     <geometry>
       <mesh filename="package://mr_robot_description/meshes/cover_1.stl" scale="0.001 0.001 0.001"/>
@@ -199,5 +198,5 @@
   </visual>
   <collision>
-    <origin rpy="0 0 0" xyz="0.006577 0.151759 -0.090182"/>
+    <origin rpy="0 0 0" xyz="0.145 -0.0 -0.09"/>
     <geometry>
       <mesh filename="package://mr_robot_description/meshes/cover_1.stl" scale="0.001 0.001 0.001"/>
@@ -207,10 +206,10 @@
 <link name="front_cover_1">
   <inertial>
-    <origin rpy="0 0 0" xyz="0.0032884224228579002 0.005869397804476428 0.029909059039267598"/>
+    <origin rpy="0 0 0" xyz="-9.965579114090684e-06 -2.2148949341271874e-16 0.025"/>
     <mass value="0.5845384389566758"/>
-    <inertia ixx="0.000123" ixy="0.0" ixz="-0.0" iyy="0.004444" iyz="0.0" izz="0.004323"/>
-  </inertial>
-  <visual>
-    <origin rpy="0 0 0" xyz="0.006577 -0.143241 -0.037682"/>
+    <inertia ixx="0.004444" ixy="-0.0" ixz="0.0" iyy="0.000123" iyz="0.0" izz="0.004323"/>
+  </inertial>
+  <visual>
+    <origin rpy="0 0 0" xyz="-0.15 0.0 -0.04"/>
     <geometry>
       <mesh filename="package://mr_robot_description/meshes/front_cover_1.stl" scale="0.001 0.001 0.001"/>
@@ -219,5 +218,5 @@
   </visual>
   <collision>
-    <origin rpy="0 0 0" xyz="0.006577 -0.143241 -0.037682"/>
+    <origin rpy="0 0 0" xyz="-0.15 0.0 -0.04"/>
     <geometry>
       <mesh filename="package://mr_robot_description/meshes/front_cover_1.stl" scale="0.001 0.001 0.001"/>
@@ -225,55 +224,105 @@
   </collision>
 </link>
-<joint name="Rigid23" type="fixed">
-  <origin rpy="0 0 0" xyz="-0.006577 -0.004259 0.040182"/>
-  <parent link="base_link"/>
-  <child link="R_motor_clamp__1__1"/>
-</joint>
-<joint name="Rigid24" type="fixed">
-  <origin rpy="0 0 0" xyz="-0.006577 -0.004259 0.040182"/>
-  <parent link="base_link"/>
-  <child link="L_motor_clamp_1"/>
-</joint>
+<link name="f_chaster_1">
+  <inertial>
+    <origin rpy="0 0 0" xyz="0.1299999999999995 -2.2819202308709316e-16 -0.01542391304347825"/>
+    <mass value="0.07562860714741833"/>
+    <inertia ixx="8e-06" ixy="-0.0" ixz="0.0" iyy="8e-06" iyz="-0.0" izz="4e-06"/>
+  </inertial>
+  <visual>
+    <origin rpy="0 0 0" xyz="0.0 -0.0 -0.035"/>
+    <geometry>
+      <mesh filename="package://mr_robot_description/meshes/f_chaster_1.stl" scale="0.001 0.001 0.001"/>
+    </geometry>
+    <material name="silver"/>
+  </visual>
+  <collision>
+    <origin rpy="0 0 0" xyz="0.0 -0.0 -0.035"/>
+    <geometry>
+      <mesh filename="package://mr_robot_description/meshes/f_chaster_1.stl" scale="0.001 0.001 0.001"/>
+    </geometry>
+  </collision>
+</link>
+<link name="b_chaster_1">
+  <inertial>
+    <origin rpy="0 0 0" xyz="-0.1299999999999995 2.304124691363434e-16 -0.015423913043478246"/>
+    <mass value="0.07562860714741829"/>
+    <inertia ixx="8e-06" ixy="0.0" ixz="-0.0" iyy="8e-06" iyz="0.0" izz="4e-06"/>
+  </inertial>
+  <visual>
+    <origin rpy="0 0 0" xyz="0.0 -0.0 -0.035"/>
+    <geometry>
+      <mesh filename="package://mr_robot_description/meshes/b_chaster_1.stl" scale="0.001 0.001 0.001"/>
+    </geometry>
+    <material name="silver"/>
+  </visual>
+  <collision>
+    <origin rpy="0 0 0" xyz="0.0 -0.0 -0.035"/>
+    <geometry>
+      <mesh filename="package://mr_robot_description/meshes/b_chaster_1.stl" scale="0.001 0.001 0.001"/>
+    </geometry>
+  </collision>
+</link>
 <joint name="Rigid25" type="fixed">
-  <origin rpy="0 0 0" xyz="-0.067712 -0.011871 0.020109"/>
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
Commit message: Changes joint axes

File: mr_robot_description/urdf/mr_robot.xacro (robot description, xacro)
@@ -3,5 +3,6 @@
 <xacro:include filename="$(find mr_robot_description)/urdf/materials.xacro" />
 <xacro:include filename="$(find mr_robot_description)/urdf/mr_robot.trans" />
-<xacro:include filename="$(find mr_robot_description)/urdf/mr_robot.gazebo" />
+<xacro:include filename="$(find mr_robot_description)/gazebo/mr_robot.gazebo" />
+<xacro:include filename="$(find mr_robot_description)/gazebo/mr_robot_plugins.gazebo" />
 <link name="base_link">
   <inertial>
@@ -278,5 +279,5 @@
   <parent link="R_motor_1"/>
   <child link="R_wheel_1"/>
-  <axis xyz="-0.0 -1.0 0.0"/>
+  <axis xyz="-0.0 1.0 0.0"/>
 </joint>
 <joint name="left_motor_joint" type="continuous">

Commit message: Changes Joint Axes

File: mr_robot_description/urdf/mr_robot.xacro (robot description, xacro)
@@ -249,5 +249,5 @@
   <parent link="R_motor_1"/>
   <child link="R_wheel_1"/>
-  <axis xyz="1.0 -0.0 0.0"/>
+  <axis xyz="1.0 0.0 0.0"/>
 </joint>
 <joint name="left_motor_joint" type="continuous">
@@ -255,5 +255,5 @@
   <parent link="L_motor_1"/>
   <child link="L_wheel_1"/>
-  <axis xyz="-1.0 0.0 -0.0"/>
+  <axis xyz="1.0 0.0 -0.0"/>
 </joint>
 <joint name="Rigid29" type="fixed">
