Commit message: Add files via upload

File: mr_robot_description/urdf/mr_robot.xacro (robot description, xacro)
@@ -3,11 +3,10 @@
 <xacro:include filename="$(find mr_robot_description)/urdf/materials.xacro" />
 <xacro:include filename="$(find mr_robot_description)/urdf/mr_robot.trans" />
-<xacro:include filename="$(find mr_robot_description)/gazebo/mr_robot.gazebo" />
-<xacro:include filename="$(find mr_robot_description)/gazebo/mr_robot_plugins.gazebo" />
+<xacro:include filename="$(find mr_robot_description)/urdf/mr_robot.gazebo" />
 <link name="base_link">
   <inertial>
-    <origin rpy="0 0 0" xyz="-0.0183828854411911 -9.351398117062208e-17 0.047762106966911216"/>
-    <mass value="0.6932522980076122"/>
-    <inertia ixx="0.007399" ixy="-0.0" ixz="0.000221" iyy="0.006915" iyz="-0.0" izz="0.013959"/>
+    <origin rpy="0 0 0" xyz="0.0008927921119775883 0.003383716812376711 0.05308182610349619"/>
+    <mass value="1.017219924928983"/>
+    <inertia ixx="0.009572" ixy="-1e-06" ixz="-1.1e-05" iyy="0.010869" iyz="-4e-06" izz="0.019625"/>
   </inertial>
   <visual>
@@ -25,161 +24,101 @@
   </collision>
 </link>
-<link name="L_motor_1">
-  <inertial>
-    <origin rpy="0 0 0" xyz="0.01549999996857043 -0.027245319885060224 -0.00017182896795726876"/>
-    <mass value="0.41014753708080764"/>
-    <inertia ixx="0.000183" ixy="0.0" ixz="0.0" iyy="5.4e-05" iyz="3e-06" izz="0.000183"/>
-  </inertial>
-  <visual>
-    <origin rpy="0 0 0" xyz="0.01275 -0.071 -0.0602"/>
-    <geometry>
-      <mesh filename="package://mr_robot_description/meshes/L_motor_1.stl" scale="0.001 0.001 0.001"/>
-    </geometry>
-    <material name="silver"/>
-  </visual>
-  <collision>
-    <origin rpy="0 0 0" xyz="0.01275 -0.071 -0.0602"/>
-    <geometry>
-      <mesh filename="package://mr_robot_description/meshes/L_motor_1.stl" scale="0.001 0.001 0.001"/>
-    </geometry>
-  </collision>
-</link>
-<link name="R_motor_1">
-  <inertial>
-    <origin rpy="0 0 0" xyz="-0.015499999968570767 0.027245319885060487 -0.00017182896795692876"/>
-    <mass value="0.41014753708080764"/>
-    <inertia ixx="0.000183" ixy="0.0" ixz="-0.0" iyy="5.4e-05" iyz="-3e-06" izz="0.000183"/>
-  </inertial>
-  <visual>
-    <origin rpy="0 0 0" xyz="-0.01775 0.071 -0.0602"/>
-    <geometry>
-      <mesh filename="package://mr_robot_description/meshes/R_motor_1.stl" scale="0.001 0.001 0.001"/>
-    </geometry>
-    <material name="silver"/>
-  </visual>
-  <collision>
-    <origin rpy="0 0 0" xyz="-0.01775 0.071 -0.0602"/>
-    <geometry>
-      <mesh filename="package://mr_robot_description/meshes/R_motor_1.stl" scale="0.001 0.001 0.001"/>
-    </geometry>
-  </collision>
-</link>
-<link name="R_wheel_1">
-  <inertial>
-    <origin rpy="0 0 0" xyz="1.7455221296147627e-14 -0.006133491954579948 -9.020562075079397e-15"/>
-    <mass value="0.33673316347081705"/>
-    <inertia ixx="0.000211" ixy="-0.0" ixz="-0.0" iyy="0.000351" iyz="0.0" izz="0.000211"/>
-  </inertial>
-  <visual>
-    <origin rpy="0 0 0" xyz="-0.00225 0.0997 -0.0534"/>
-    <geometry>
-      <mesh filename="package://mr_robot_description/meshes/R_wheel_1.stl" scale="0.001 0.001 0.001"/>
-    </geometry>
-    <material name="silver"/>
-  </visual>
-  <collision>
-    <origin rpy="0 0 0" xyz="-0.00225 0.0997 -0.0534"/>
-    <geometry>
-      <mesh filename="package://mr_robot_description/meshes/R_wheel_1.stl" scale="0.001 0.001 0.001"/>
-    </geometry>
-  </collision>
-</link>
-<link name="L_wheel_1">
-  <inertial>
-    <origin rpy="0 0 0" xyz="-1.705927066275592e-14 0.006133491954580114 -1.004057947895376e-14"/>
+<link name="r_wheel_1">
+  <inertial>
+    <origin rpy="0 0 0" xyz="1.974679100791299e-14 -0.002525912487815571 -1.9068080447937064e-14"/>
+    <mass value="0.17056892200116738"/>
+    <inertia ixx="0.000171" ixy="-0.0" ixz="-0.0" iyy="0.000291" iyz="0.0" izz="0.000171"/>
+  </inertial>
+  <visual>
+    <origin rpy="0 0 0" xyz="-0.00225 0.0962 -0.0534"/>
+    <geometry>
+      <mesh filename="package://mr_robot_description/meshes/r_wheel_1.stl" scale="0.001 0.001 0.001"/>
+    </geometry>
+    <material name="silver"/>
+  </visual>
+  <collision>
+    <origin rpy="0 0 0" xyz="-0.00225 0.0962 -0.0534"/>
+    <geometry>
+      <mesh filename="package://mr_robot_description/meshes/r_wheel_1.stl" scale="0.001 0.001 0.001"/>
+    </geometry>
+  </collision>
+</link>
+<link name="l_wheel_1">
+  <inertial>
+    <origin rpy="0 0 0" xyz="-1.6607375197263963e-14 0.006133491954579892 -9.936496070395151e-15"/>
     <mass value="0.33673316347081705"/>
     <inertia ixx="0.000211" ixy="-0.0" ixz="0.0" iyy="0.000351" iyz="-0.0" izz="0.000211"/>
   </inertial>
   <visual>
-    <origin rpy="0 0 0" xyz="-0.00275 -0.0997 -0.0534"/>
-    <geometry>
-      <mesh filename="package://mr_robot_description/meshes/L_wheel_1.stl" scale="0.001 0.001 0.001"/>
-    </geometry>
-    <material name="silver"/>
-  </visual>
-  <collision>
-    <origin rpy="0 0 0" xyz="-0.00275 -0.0997 -0.0534"/>
-    <geometry>
-      <mesh filename="package://mr_robot_description/meshes/L_wheel_1.stl" scale="0.001 0.001 0.001"/>
-    </geometry>
-  </collision>
-</link>
-<link name="L_motor_clamp_1">
-  <inertial>
-    <origin rpy="0 0 0" xyz="-8.07643882327902e-15 0.0665047179820893 0.0107653911894319"/>
-    <mass value="0.019214264346508234"/>
-    <inertia ixx="4e-06" ixy="-0.0" ixz="-0.0" iyy="7e-06" iyz="-1e-06" izz="4e-06"/>
-  </inertial>
-  <visual>
-    <origin rpy="0 0 0" xyz="-0.0025 0.0 -0.04"/>
-    <geometry>
-      <mesh filename="package://mr_robot_description/meshes/L_motor_clamp_1.stl" scale="0.001 0.001 0.001"/>
-    </geometry>
-    <material name="silver"/>
-  </visual>
-  <collision>
-    <origin rpy="0 0 0" xyz="-0.0025 0.0 -0.04"/>
-    <geometry>
-      <mesh filename="package://mr_robot_description/meshes/L_motor_clamp_1.stl" scale="0.001 0.001 0.001"/>
-    </geometry>
-  </collision>
-</link>
-<link name="R_motor_clamp_1">
-  <inertial>
-    <origin rpy="0 0 0" xyz="8.05995895025724e-15 -0.06650471798208926 0.010765391189432517"/>
-    <mass value="0.019214264346508234"/>
-    <inertia ixx="4e-06" ixy="-0.0" ixz="0.0" iyy="7e-06" iyz="1e-06" izz="4e-06"/>
-  </inertial>
-  <visual>
-    <origin rpy="0 0 0" xyz="-0.0025 0.0 -0.04"/>
-    <geometry>
-      <mesh filename="package://mr_robot_description/meshes/R_motor_clamp_1.stl" scale="0.001 0.001 0.001"/>
-    </geometry>
-    <material name="silver"/>
-  </visual>
-  <collision>
-    <origin rpy="0 0 0" xyz="-0.0025 0.0 -0.04"/>
-    <geometry>
-      <mesh filename="package://mr_robot_description/meshes/R_motor_clamp_1.stl" scale="0.001 0.001 0.001"/>
-    </geometry>
-  </collision>
-</link>
-<link name="motor_driver_1">
-  <inertial>
-    <origin rpy="0 0 0" xyz="-0.043295829595900504 0.0008362290865504151 0.00719092005623221"/>
-    <mass value="0.016082198290596435"/>
-    <inertia ixx="2e-06" ixy="0.0" ixz="-1e-06" iyy="3e-06" iyz="0.0" izz="4e-06"/>
-  </inertial>
-  <visual>
-    <origin rpy="0 0 0" xyz="-0.0025 0.0 -0.04"/>
-    <geometry>
-      <mesh filename="package://mr_robot_description/meshes/motor_driver_1.stl" scale="0.001 0.001 0.001"/>
-    </geometry>
-    <material name="silver"/>
-  </visual>
-  <collision>
-    <origin rpy="0 0 0" xyz="-0.0025 0.0 -0.04"/>
-    <geometry>
-      <mesh filename="package://mr_robot_description/meshes/motor_driver_1.stl" scale="0.001 0.001 0.001"/>
-    </geometry>
-  </collision>
-</link>
-<link name="battery_1">
-  <inertial>
-    <origin rpy="0 0 0" xyz="0.03999999999999985 0.0009562154241530774 0.017000000000000022"/>
-    <mass value="0.49636285277615166"/>
-    <inertia ixx="0.000509" ixy="-0.0" ixz="0.0" iyy="6.9e-05" iyz="-0.0" izz="0.000483"/>
-  </inertial>
-  <visual>
-    <origin rpy="0 0 0" xyz="-0.0025 0.0 -0.04"/>
-    <geometry>
-      <mesh filename="package://mr_robot_description/meshes/battery_1.stl" scale="0.001 0.001 0.001"/>
-    </geometry>
-    <material name="silver"/>
-  </visual>
-  <collision>
-    <origin rpy="0 0 0" xyz="-0.0025 0.0 -0.04"/>
-    <geometry>
-      <mesh filename="package://mr_robot_description/meshes/battery_1.stl" scale="0.001 0.001 0.001"/>
+    <origin rpy="0 0 0" xyz="-0.00275 -0.1032 -0.0534"/>
+    <geometry>
+      <mesh filename="package://mr_robot_description/meshes/l_wheel_1.stl" scale="0.001 0.001 0.001"/>
+    </geometry>
+    <material name="silver"/>
+  </visual>
+  <collision>
+    <origin rpy="0 0 0" xyz="-0.00275 -0.1032 -0.0534"/>
+    <geometry>
+      <mesh filename="package://mr_robot_description/meshes/l_wheel_1.stl" scale="0.001 0.001 0.001"/>
+    </geometry>
+  </collision>
+</link>
+<link name="lidar_cover_1">
+  <inertial>
+    <origin rpy="0 0 0" xyz="-0.13381670754509806 -0.002195336861350322 -0.11800000000000005"/>
+    <mass value="0.31059474429759854"/>
+    <inertia ixx="0.000448" ixy="-3e-06" ixz="-0.0" iyy="0.000606" iyz="0.0" izz="0.001054"/>
+  </inertial>
+  <visual>
+    <origin rpy="0 0 0" xyz="-0.209625 -0.007 -0.225"/>
+    <geometry>
+      <mesh filename="package://mr_robot_description/meshes/lidar_cover_1.stl" scale="0.001 0.001 0.001"/>
+    </geometry>
+    <material name="silver"/>
+  </visual>
+  <collision>
+    <origin rpy="0 0 0" xyz="-0.209625 -0.007 -0.225"/>
+    <geometry>
+      <mesh filename="package://mr_robot_description/meshes/lidar_cover_1.stl" scale="0.001 0.001 0.001"/>
+    </geometry>
+  </collision>
+</link>
+<link name="l_tyre_wall_1">
+  <inertial>
+    <origin rpy="0 0 0" xyz="-0.002842639819893089 0.02036548235514131 -0.01397208252909686"/>
+    <mass value="0.5799187471048897"/>
+    <inertia ixx="0.000566" ixy="-5e-06" ixz="-2e-06" iyy="0.001977" iyz="1.5e-05" izz="0.002185"/>
+  </inertial>
+  <visual>
+    <origin rpy="0 0 0" xyz="-0.0025 -0.07525 -0.08"/>
+    <geometry>
+      <mesh filename="package://mr_robot_description/meshes/l_tyre_wall_1.stl" scale="0.001 0.001 0.001"/>
+    </geometry>
+    <material name="silver"/>
+  </visual>
+  <collision>
+    <origin rpy="0 0 0" xyz="-0.0025 -0.07525 -0.08"/>
+    <geometry>
+      <mesh filename="package://mr_robot_description/meshes/l_tyre_wall_1.stl" scale="0.001 0.001 0.001"/>
+    </geometry>
+  </collision>
+</link>
+<link name="r_tyre_wall_1">
+  <inertial>
+    <origin rpy="0 0 0" xyz="-0.002842639819893113 -0.02036548235514124 -0.01397208252909593"/>
+    <mass value="0.5799187471048897"/>
+    <inertia ixx="0.000566" ixy="5e-06" ixz="-2e-06" iyy="0.001977" iyz="-1.5e-05" izz="0.002185"/>
+  </inertial>
+  <visual>
+    <origin rpy="0 0 0" xyz="-0.0025 0.06825 -0.08"/>
+    <geometry>
+      <mesh filename="package://mr_robot_description/meshes/r_tyre_wall_1.stl" scale="0.001 0.001 0.001"/>
+    </geometry>
+    <material name="silver"/>
+  </visual>
+  <collision>
+    <origin rpy="0 0 0" xyz="-0.0025 0.06825 -0.08"/>
+    <geometry>
+      <mesh filename="package://mr_robot_description/meshes/r_tyre_wall_1.stl" scale="0.001 0.001 0.001"/>
     </geometry>
   </collision>
@@ -187,10 +126,10 @@
 <link name="cover_1">
   <inertial>
-    <origin rpy="0 0 0" xyz="0.143794391136608 -0.00013907701861727573 0.0024942607758274143"/>
-    <mass value="3.0449746602441645"/>
-    <inertia ixx="0.021423" ixy="-1e-05" ixz="3e-06" iyy="0.025731" iyz="0.0" izz="0.047142"/>
-  </inertial>
-  <visual>
-    <origin rpy="0 0 0" xyz="0.145 -0.0 -0.09"/>
+    <origin rpy="0 0 0" xyz="0.13333687933642632 -0.0004534984394031767 0.0024952118809939416"/>
+    <mass value="2.5548768748457116"/>
+    <inertia ixx="0.02109" ixy="6.7e-05" ixz="2e-06" iyy="0.021151" iyz="-0.0" izz="0.04223"/>
+  </inertial>
+  <visual>
+    <origin rpy="0 0 0" xyz="0.15 -0.0035 -0.1"/>
     <geometry>
       <mesh filename="package://mr_robot_description/meshes/cover_1.stl" scale="0.001 0.001 0.001"/>
@@ -199,5 +138,5 @@
   </visual>
   <collision>
-    <origin rpy="0 0 0" xyz="0.145 -0.0 -0.09"/>
+    <origin rpy="0 0 0" xyz="0.15 -0.0035 -0.1"/>
     <geometry>
       <mesh filename="package://mr_robot_description/meshes/cover_1.stl" scale="0.001 0.001 0.001"/>
@@ -205,125 +144,60 @@
   </collision>
 </link>
-<link name="front_cover_1">
-  <inertial>
-    <origin rpy="0 0 0" xyz="-9.965579114090684e-06 -2.2148949341271874e-16 0.025"/>
-    <mass value="0.5845384389566758"/>
-    <inertia ixx="0.004444" ixy="-0.0" ixz="0.0" iyy="0.000123" iyz="0.0" izz="0.004323"/>
-  </inertial>
-  <visual>
-    <origin rpy="0 0 0" xyz="-0.15 0.0 -0.04"/>
-    <geometry>
-      <mesh filename="package://mr_robot_description/meshes/front_cover_1.stl" scale="0.001 0.001 0.001"/>
-    </geometry>
-    <material name="silver"/>
-  </visual>
-  <collision>
-    <origin rpy="0 0 0" xyz="-0.15 0.0 -0.04"/>
-    <geometry>
-      <mesh filename="package://mr_robot_description/meshes/front_cover_1.stl" scale="0.001 0.001 0.001"/>
-    </geometry>
-  </collision>
-</link>
-<link name="f_chaster_1">
-  <inertial>
-    <origin rpy="0 0 0" xyz="0.1299999999999995 -2.2819202308709316e-16 -0.01542391304347825"/>
-    <mass value="0.07562860714741833"/>
-    <inertia ixx="8e-06" ixy="-0.0" ixz="0.0" iyy="8e-06" iyz="-0.0" izz="4e-06"/>
-  </inertial>
-  <visual>
-    <origin rpy="0 0 0" xyz="0.0 -0.0 -0.035"/>
-    <geometry>
-      <mesh filename="package://mr_robot_description/meshes/f_chaster_1.stl" scale="0.001 0.001 0.001"/>
-    </geometry>
-    <material name="silver"/>
-  </visual>
-  <collision>
-    <origin rpy="0 0 0" xyz="0.0 -0.0 -0.035"/>
-    <geometry>
-      <mesh filename="package://mr_robot_description/meshes/f_chaster_1.stl" scale="0.001 0.001 0.001"/>
-    </geometry>
-  </collision>
-</link>
-<link name="b_chaster_1">
-  <inertial>
-    <origin rpy="0 0 0" xyz="-0.1299999999999995 2.304124691363434e-16 -0.015423913043478246"/>
-    <mass value="0.07562860714741829"/>
-    <inertia ixx="8e-06" ixy="0.0" ixz="-0.0" iyy="8e-06" iyz="0.0" izz="4e-06"/>
-  </inertial>
-  <visual>
-    <origin rpy="0 0 0" xyz="0.0 -0.0 -0.035"/>
-    <geometry>
-      <mesh filename="package://mr_robot_description/meshes/b_chaster_1.stl" scale="0.001 0.001 0.001"/>
-    </geometry>
-    <material name="silver"/>
-  </visual>
-  <collision>
-    <origin rpy="0 0 0" xyz="0.0 -0.0 -0.035"/>
-    <geometry>
-      <mesh filename="package://mr_robot_description/meshes/b_chaster_1.stl" scale="0.001 0.001 0.001"/>
-    </geometry>
-  </collision>
-</link>
-<joint name="Rigid25" type="fixed">
-  <origin rpy="0 0 0" xyz="-0.01525 0.071 0.0202"/>
-  <parent link="L_motor_clamp_1"/>
-  <child link="L_motor_1"/>
-</joint>
-<joint name="Rigid26" type="fixed">
-  <origin rpy="0 0 0" xyz="0.01525 -0.071 0.0202"/>
-  <parent link="R_motor_clamp_1"/>
-  <child link="R_motor_1"/>
-</joint>
+<link name="ydlidar_x4_v1_1">
+  <inertial>
+    <origin rpy="0 0 0" xyz="-0.048294448377836835 -2.8189256484623115e-17 0.06720114222279103"/>
+    <mass value="1.1515616542314233"/>
+    <inertia ixx="0.000489" ixy="-0.0" ixz="-0.000148" iyy="0.000861" iyz="0.0" izz="0.000987"/>
+  </inertial>
+  <visual>
+    <origin rpy="0 0 0" xyz="-0.144813 -0.0035 -0.04"/>
+    <geometry>
+      <mesh filename="package://mr_robot_description/meshes/ydlidar_x4_v1_1.stl" scale="0.001 0.001 0.001"/>
+    </geometry>
+    <material name="silver"/>
+  </visual>
+  <collision>
+    <origin rpy="0 0 0" xyz="-0.144813 -0.0035 -0.04"/>
+    <geometry>
+      <mesh filename="package://mr_robot_description/meshes/ydlidar_x4_v1_1.stl" scale="0.001 0.001 0.001"/>
+    </geometry>
+  </collision>
+</link>
 <joint name="right_motor_joint" type="continuous">
-  <origin rpy="0 0 0" xyz="-0.0155 -0.0287 -0.0068"/>
-  <parent link="R_motor_1"/>
-  <child link="R_wheel_1"/>
-  <axis xyz="-0.0 1.0 0.0"/>
+  <origin rpy="0 0 0" xyz="0.00225 -0.0962 0.0534"/>
+  <parent link="base_link"/>
+  <child link="r_wheel_1"/>
+  <axis xyz="-0.0 -1.0 0.0"/>
 </joint>
 <joint name="left_motor_joint" type="continuous">
-  <origin rpy="0 0 0" xyz="0.0155 0.0287 -0.0068"/>
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