Commit message: Add files via upload
reduced joints

File: mr_robot_description/urdf/mr_robot.xacro (robot description, xacro)
@@ -6,7 +6,7 @@
 <link name="base_link">
   <inertial>
-    <origin rpy="0 0 0" xyz="0.0008927921119775883 0.003383716812376711 0.05308182610349619"/>
-    <mass value="1.017219924928983"/>
-    <inertia ixx="0.009572" ixy="-1e-06" ixz="-1.1e-05" iyy="0.010869" iyz="-4e-06" izz="0.019625"/>
+    <origin rpy="0 0 0" xyz="-0.00101458512283434 -0.0007739653318165107 0.06722998744578039"/>
+    <mass value="11.545387094155112"/>
+    <inertia ixx="0.101768" ixy="-1.2e-05" ixz="0.000834" iyy="0.108037" iyz="4.2e-05" izz="0.192707"/>
   </inertial>
   <visual>
@@ -24,180 +24,80 @@
   </collision>
 </link>
-<link name="r_wheel_1">
+<link name="r_tyre_1">
   <inertial>
-    <origin rpy="0 0 0" xyz="1.974679100791299e-14 -0.002525912487815571 -1.9068080447937064e-14"/>
-    <mass value="0.17056892200116738"/>
-    <inertia ixx="0.000171" ixy="-0.0" ixz="-0.0" iyy="0.000291" iyz="0.0" izz="0.000171"/>
+    <origin rpy="0 0 0" xyz="9.682659047986764e-08 -0.002525549104224978 -5.1894622932202594e-08"/>
+    <mass value="1.4397484276442625"/>
+    <inertia ixx="0.00144" ixy="-0.0" ixz="-0.0" iyy="0.00246" iyz="0.0" izz="0.00144"/>
   </inertial>
   <visual>
-    <origin rpy="0 0 0" xyz="-0.00225 0.0962 -0.0534"/>
+    <origin rpy="0 0 0" xyz="0.003445 0.10058 -0.052283"/>
     <geometry>
-      <mesh filename="package://mr_robot_description/meshes/r_wheel_1.stl" scale="0.001 0.001 0.001"/>
+      <mesh filename="package://mr_robot_description/meshes/r_tyre_1.stl" scale="0.001 0.001 0.001"/>
     </geometry>
     <material name="silver"/>
   </visual>
   <collision>
-    <origin rpy="0 0 0" xyz="-0.00225 0.0962 -0.0534"/>
+    <origin rpy="0 0 0" xyz="0.003445 0.10058 -0.052283"/>
     <geometry>
-      <mesh filename="package://mr_robot_description/meshes/r_wheel_1.stl" scale="0.001 0.001 0.001"/>
+      <mesh filename="package://mr_robot_description/meshes/r_tyre_1.stl" scale="0.001 0.001 0.001"/>
     </geometry>
   </collision>
 </link>
-<link name="l_wheel_1">
+<link name="l_tyre_1">
   <inertial>
-    <origin rpy="0 0 0" xyz="-1.6607375197263963e-14 0.006133491954579892 -9.936496070395151e-15"/>
-    <mass value="0.33673316347081705"/>
-    <inertia ixx="0.000211" ixy="-0.0" ixz="0.0" iyy="0.000351" iyz="-0.0" izz="0.000211"/>
+    <origin rpy="0 0 0" xyz="9.682664276963737e-08 0.0025262758714060807 -5.18946233832307e-08"/>
+    <mass value="1.4397484276442625"/>
+    <inertia ixx="0.00144" ixy="-0.0" ixz="0.0" iyy="0.00246" iyz="-0.0" izz="0.00144"/>
   </inertial>
   <visual>
-    <origin rpy="0 0 0" xyz="-0.00275 -0.1032 -0.0534"/>
+    <origin rpy="0 0 0" xyz="0.003445 -0.09882 -0.052283"/>
     <geometry>
-      <mesh filename="package://mr_robot_description/meshes/l_wheel_1.stl" scale="0.001 0.001 0.001"/>
+      <mesh filename="package://mr_robot_description/meshes/l_tyre_1.stl" scale="0.001 0.001 0.001"/>
     </geometry>
     <material name="silver"/>
   </visual>
   <collision>
-    <origin rpy="0 0 0" xyz="-0.00275 -0.1032 -0.0534"/>
+    <origin rpy="0 0 0" xyz="0.003445 -0.09882 -0.052283"/>
     <geometry>
-      <mesh filename="package://mr_robot_description/meshes/l_wheel_1.stl" scale="0.001 0.001 0.001"/>
+      <mesh filename="package://mr_robot_description/meshes/l_tyre_1.stl" scale="0.001 0.001 0.001"/>
     </geometry>
   </collision>
 </link>
-<link name="lidar_cover_1">
+<link name="lidar_1">
   <inertial>
-    <origin rpy="0 0 0" xyz="-0.13381670754509806 -0.002195336861350322 -0.11800000000000005"/>
-    <mass value="0.31059474429759854"/>
-    <inertia ixx="0.000448" ixy="-3e-06" ixz="-0.0" iyy="0.000606" iyz="0.0" izz="0.001054"/>
+    <origin rpy="0 0 0" xyz="-0.006349391522619652 0.0008793633835904074 -0.002389798737942095"/>
+    <mass value="1.1515616542314233"/>
+    <inertia ixx="0.000489" ixy="-0.0" ixz="-0.000148" iyy="0.000861" iyz="0.0" izz="0.000987"/>
   </inertial>
   <visual>
-    <origin rpy="0 0 0" xyz="-0.209625 -0.007 -0.225"/>
+    <origin rpy="0 0 0" xyz="-0.0967 0.001759 -0.108682"/>
     <geometry>
-      <mesh filename="package://mr_robot_description/meshes/lidar_cover_1.stl" scale="0.001 0.001 0.001"/>
+      <mesh filename="package://mr_robot_description/meshes/lidar_1.stl" scale="0.001 0.001 0.001"/>
     </geometry>
     <material name="silver"/>
   </visual>
   <collision>
-    <origin rpy="0 0 0" xyz="-0.209625 -0.007 -0.225"/>
+    <origin rpy="0 0 0" xyz="-0.0967 0.001759 -0.108682"/>
     <geometry>
-      <mesh filename="package://mr_robot_description/meshes/lidar_cover_1.stl" scale="0.001 0.001 0.001"/>
+      <mesh filename="package://mr_robot_description/meshes/lidar_1.stl" scale="0.001 0.001 0.001"/>
     </geometry>
   </collision>
 </link>
-<link name="l_tyre_wall_1">
-  <inertial>
-    <origin rpy="0 0 0" xyz="-0.002842639819893089 0.02036548235514131 -0.01397208252909686"/>
-    <mass value="0.5799187471048897"/>
-    <inertia ixx="0.000566" ixy="-5e-06" ixz="-2e-06" iyy="0.001977" iyz="1.5e-05" izz="0.002185"/>
-  </inertial>
-  <visual>
-    <origin rpy="0 0 0" xyz="-0.0025 -0.07525 -0.08"/>
-    <geometry>
-      <mesh filename="package://mr_robot_description/meshes/l_tyre_wall_1.stl" scale="0.001 0.001 0.001"/>
-    </geometry>
-    <material name="silver"/>
-  </visual>
-  <collision>
-    <origin rpy="0 0 0" xyz="-0.0025 -0.07525 -0.08"/>
-    <geometry>
-      <mesh filename="package://mr_robot_description/meshes/l_tyre_wall_1.stl" scale="0.001 0.001 0.001"/>
-    </geometry>
-  </collision>
-</link>
-<link name="r_tyre_wall_1">
-  <inertial>
-    <origin rpy="0 0 0" xyz="-0.002842639819893113 -0.02036548235514124 -0.01397208252909593"/>
-    <mass value="0.5799187471048897"/>
-    <inertia ixx="0.000566" ixy="5e-06" ixz="-2e-06" iyy="0.001977" iyz="-1.5e-05" izz="0.002185"/>
-  </inertial>
-  <visual>
-    <origin rpy="0 0 0" xyz="-0.0025 0.06825 -0.08"/>
-    <geometry>
-      <mesh filename="package://mr_robot_description/meshes/r_tyre_wall_1.stl" scale="0.001 0.001 0.001"/>
-    </geometry>
-    <material name="silver"/>
-  </visual>
-  <collision>
-    <origin rpy="0 0 0" xyz="-0.0025 0.06825 -0.08"/>
-    <geometry>
-      <mesh filename="package://mr_robot_description/meshes/r_tyre_wall_1.stl" scale="0.001 0.001 0.001"/>
-    </geometry>
-  </collision>
-</link>
-<link name="cover_1">
-  <inertial>
-    <origin rpy="0 0 0" xyz="0.13333687933642632 -0.0004534984394031767 0.0024952118809939416"/>
-    <mass value="2.5548768748457116"/>
-    <inertia ixx="0.02109" ixy="6.7e-05" ixz="2e-06" iyy="0.021151" iyz="-0.0" izz="0.04223"/>
-  </inertial>
-  <visual>
-    <origin rpy="0 0 0" xyz="0.15 -0.0035 -0.1"/>
-    <geometry>
-      <mesh filename="package://mr_robot_description/meshes/cover_1.stl" scale="0.001 0.001 0.001"/>
-    </geometry>
-    <material name="silver"/>
-  </visual>
-  <collision>
-    <origin rpy="0 0 0" xyz="0.15 -0.0035 -0.1"/>
-    <geometry>
-      <mesh filename="package://mr_robot_description/meshes/cover_1.stl" scale="0.001 0.001 0.001"/>
-    </geometry>
-  </collision>
-</link>
-<link name="ydlidar_x4_v1_1">
-  <inertial>
-    <origin rpy="0 0 0" xyz="-0.048294448377836835 -2.8189256484623115e-17 0.06720114222279103"/>
-    <mass value="1.1515616542314233"/>
-    <inertia ixx="0.000489" ixy="-0.0" ixz="-0.000148" iyy="0.000861" iyz="0.0" izz="0.000987"/>
-  </inertial>
-  <visual>
-    <origin rpy="0 0 0" xyz="-0.144813 -0.0035 -0.04"/>
-    <geometry>
-      <mesh filename="package://mr_robot_description/meshes/ydlidar_x4_v1_1.stl" scale="0.001 0.001 0.001"/>
-    </geometry>
-    <material name="silver"/>
-  </visual>
-  <collision>
-    <origin rpy="0 0 0" xyz="-0.144813 -0.0035 -0.04"/>
-    <geometry>
-      <mesh filename="package://mr_robot_description/meshes/ydlidar_x4_v1_1.stl" scale="0.001 0.001 0.001"/>
-    </geometry>
-  </collision>
-</link>
-<joint name="right_motor_joint" type="continuous">
-  <origin rpy="0 0 0" xyz="0.00225 -0.0962 0.0534"/>
+<joint name="R_Rev" type="continuous">
+  <origin rpy="0 0 0" xyz="-0.003445 -0.10058 0.052283"/>
   <parent link="base_link"/>
-  <child link="r_wheel_1"/>
-  <axis xyz="-0.0 -1.0 0.0"/>
+  <child link="r_tyre_1"/>
+  <axis xyz="-0.0 -1.0 -0.0"/>
 </joint>
-<joint name="left_motor_joint" type="continuous">
-  <origin rpy="0 0 0" xyz="0.00275 0.1032 0.0534"/>
+<joint name="L_Rev" type="continuous">
+  <origin rpy="0 0 0" xyz="-0.003445 0.09882 0.052283"/>
   <parent link="base_link"/>
-  <child link="l_wheel_1"/>
-  <axis xyz="0.0 1.0 -0.0"/>
+  <child link="l_tyre_1"/>
+  <axis xyz="0.0 1.0 0.0"/>
 </joint>
-<joint name="Rigid48" type="fixed">
-  <origin rpy="0 0 0" xyz="0.064812 0.0035 0.185"/>
-  <parent link="ydlidar_x4_v1_1"/>
-  <child link="lidar_cover_1"/>
-</joint>
-<joint name="Rigid51" type="fixed">
-  <origin rpy="0 0 0" xyz="0.0025 0.07525 0.08"/>
+<joint name="lidar_fixed" type="fixed">
+  <origin rpy="0 0 0" xyz="0.0967 -0.001759 0.108682"/>
   <parent link="base_link"/>
-  <child link="l_tyre_wall_1"/>
-</joint>
-<joint name="Rigid52" type="fixed">
-  <origin rpy="0 0 0" xyz="0.0025 -0.06825 0.08"/>
-  <parent link="base_link"/>
-  <child link="r_tyre_wall_1"/>
-</joint>
-<joint name="Rigid53" type="fixed">
-  <origin rpy="0 0 0" xyz="-0.15 0.0035 0.1"/>
-  <parent link="base_link"/>
-  <child link="cover_1"/>
-</joint>
-<joint name="Rigid55" type="fixed">
-  <origin rpy="0 0 0" xyz="0.144813 0.0035 0.04"/>
-  <parent link="base_link"/>
-  <child link="ydlidar_x4_v1_1"/>
+  <child link="lidar_1"/>
 </joint>
 </robot>

Commit message: Corrects wheel joint names & Corrects wheel joint axis

File: mr_robot_description/urdf/mr_robot.xacro (robot description, xacro)
@@ -3,5 +3,6 @@
 <xacro:include filename="$(find mr_robot_description)/urdf/materials.xacro" />
 <xacro:include filename="$(find mr_robot_description)/urdf/mr_robot.trans" />
-<xacro:include filename="$(find mr_robot_description)/urdf/mr_robot.gazebo" />
+<xacro:include filename="$(find mr_robot_description)/gazebo/mr_robot.gazebo" />
+<xacro:include filename="$(find mr_robot_description)/gazebo/mr_robot_plugins.gazebo" />
 <link name="base_link">
   <inertial>
@@ -84,11 +85,11 @@
   </collision>
 </link>
-<joint name="R_Rev" type="continuous">
+<joint name="right_motor_joint" type="continuous">
   <origin rpy="0 0 0" xyz="-0.003445 -0.10058 0.052283"/>
   <parent link="base_link"/>
   <child link="r_tyre_1"/>
-  <axis xyz="-0.0 -1.0 -0.0"/>
+  <axis xyz="-0.0 1.0 -0.0"/>
 </joint>
-<joint name="L_Rev" type="continuous">
+<joint name="left_motor_joint" type="continuous">
   <origin rpy="0 0 0" xyz="-0.003445 0.09882 0.052283"/>
   <parent link="base_link"/>

Commit message: Added camera plugin

File: mr_robot_description/urdf/mr_robot.xacro (robot description, xacro)
@@ -102,3 +102,30 @@
   <child link="lidar_1"/>
 </joint>
+ <xacro:property name="camera_link" value="0.05" /> <!-- Size of square 'camera' box -->
+  <joint name="camera_joint" type="fixed">
+  <origin rpy="0 0 0" xyz="0.0967 -0.001759 0.163682"/>
+  <parent link="base_link"/>
+  <child link="camera_link"/>
+</joint>
+  <!-- Camera -->
+  <link name="camera_link">
+    <collision>
+      <origin xyz="0 0 0" rpy="0 0 0"/>
+      <geometry>
+    <box size="${camera_link} ${camera_link} ${camera_link}"/>
+      </geometry>
+    </collision>
+    <visual>
+      <origin xyz="0 0 0" rpy="0 0 0"/>
+      <geometry>
+    <box size="${camera_link} ${camera_link} ${camera_link}"/>
+      </geometry>
+      <material name="red"/>
+    </visual>
+    <inertial>
+      <mass value="1e-5" />
+      <origin xyz="0 0 0" rpy="0 0 0"/>
+      <inertia ixx="1e-6" ixy="0" ixz="0" iyy="1e-6" iyz="0" izz="1e-6" />
+    </inertial>
+  </link>
 </robot>

Commit message: add_point_clout

File: mr_robot_description/urdf/mr_robot.xacro (robot description, xacro)
@@ -5,4 +5,6 @@
 <xacro:include filename="$(find mr_robot_description)/gazebo/mr_robot.gazebo" />
 <xacro:include filename="$(find mr_robot_description)/gazebo/mr_robot_plugins.gazebo" />
+<xacro:property name="camera_depth_frame" value="0.05" />
+<xacro:property name="camera_link" value="0.05" />
 <link name="base_link">
   <inertial>
@@ -85,4 +87,46 @@
   </collision>
 </link>
+<link name="camera_depth_frame">
+    <collision>
+      <origin xyz="0 0 0" rpy="0 0 7.85"/>
+      <geometry>
+        <mesh filename="package://mr_robot_description/meshes/kinect.stl" scale="0.005 0.005 0.005"/>
+      </geometry>
+    </collision>
+    <visual>
+      <origin xyz="0 0 0" rpy="0 0 7.85"/>
+      <geometry>
+    <!--<box size="${kinect_link} ${kinect_link} ${kinect_link}"/>-->
+        <mesh filename="package://mr_robot_description/meshes/kinect.stl" scale="0.005 0.005 0.005"/>
+      </geometry>
+      <material name="red"/>
+    </visual>
+    <inertial>
+      <mass value="1e-5" />
+      <origin xyz="0 0 0" rpy="0 0 7.85"/>
+      <inertia ixx="1e-6" ixy="0" ixz="0" iyy="1e-6" iyz="0" izz="1e-6" />
+    </inertial>
+  </link>
+ <!-- Camera -->
+   <link name="camera_link">
+    <collision>
+      <origin xyz="0 0 0" rpy="0 0 0"/>
+      <geometry>
+    <box size="${camera_link} ${camera_link} ${camera_link}"/>
+        </geometry>
+    </collision>
+    <visual>
+      <origin xyz="0 0 0" rpy="0 0 0"/>
+      <geometry>
+    <box size="${camera_link} ${camera_link} ${camera_link}"/>
+      </geometry>
+      <material name="red"/>
+    </visual>
+    <inertial>
+      <mass value="1e-5" />
+      <origin xyz="0 0 0" rpy="0 0 0"/>
+      <inertia ixx="1e-6" ixy="0" ixz="0" iyy="1e-6" iyz="0" izz="1e-6" />
+    </inertial>
+  </link>
 <joint name="right_motor_joint" type="continuous">
   <origin rpy="0 0 0" xyz="-0.003445 -0.10058 0.052283"/>
@@ -102,3 +146,13 @@
   <child link="lidar_1"/>
 </joint>
+<joint name="camera_joint" type="fixed">
+  <origin rpy="0 0 0" xyz="0.0967 -0.001759 0.163682"/>
+  <parent link="base_link"/>
+  <child link="camera_link"/>
+</joint>
+<joint name="depth_joint" type="fixed">
+  <origin rpy="0 0 0" xyz="0.0967 -0.001759 0.143682"/>
+  <parent link="base_link"/>
+  <child link="camera_depth_frame"/>
+</joint>
 </robot>

Commit message: laser_frame

File: mr_robot_description/urdf/mr_robot.xacro (robot description, xacro)
@@ -65,5 +65,5 @@
   </collision>
 </link>
-<link name="lidar_1">
+<link name="laser_frame">
   <inertial>
     <origin rpy="0 0 0" xyz="-0.006349391522619652 0.0008793633835904074 -0.002389798737942095"/>

Commit message: laser_frame

File: mr_robot_description/urdf/mr_robot.xacro (robot description, xacro)
@@ -100,5 +100,5 @@
   <origin rpy="0 0 0" xyz="0.0967 -0.001759 0.108682"/>
   <parent link="base_link"/>
-  <child link="lidar_1"/>
+  <child link="lidar_frame"/>
 </joint>
 </robot>

Commit message: laser_frame

File: mr_robot_description/urdf/mr_robot.xacro (robot description, xacro)
@@ -100,5 +100,5 @@
   <origin rpy="0 0 0" xyz="0.0967 -0.001759 0.108682"/>
   <parent link="base_link"/>
-  <child link="lidar_frame"/>
+  <child link="laser_frame"/>
 </joint>
 </robot>

Commit message: fix 1

File: mr_robot_description/urdf/mr_robot.xacro (robot description, xacro)
@@ -101,4 +101,5 @@
   <parent link="base_link"/>
   <child link="laser_frame"/>
+  <axis xyz="-0.0 1.0 -0.0"/>
 </joint>
 </robot>

Commit message: fix2

File: mr_robot_description/urdf/mr_robot.xacro (robot description, xacro)
@@ -101,5 +101,4 @@
   <parent link="base_link"/>
   <child link="laser_frame"/>
-  <axis xyz="-0.0 1.0 -0.0"/>
 </joint>
 </robot>

Commit message: changed to lidar_1

File: mr_robot_description/urdf/mr_robot.xacro (robot description, xacro)
@@ -65,5 +65,5 @@
   </collision>
 </link>
-<link name="laser_frame">
+<link name="lidar_1">
   <inertial>
     <origin rpy="0 0 0" xyz="-0.006349391522619652 0.0008793633835904074 -0.002389798737942095"/>
@@ -100,5 +100,5 @@
   <origin rpy="0 0 0" xyz="0.0967 -0.001759 0.108682"/>
   <parent link="base_link"/>
-  <child link="laser_frame"/>
+  <child link="lidar_1"/>
 </joint>
 </robot>

Commit message: mapping added

File: mr_robot_description/urdf/mr_robot.xacro (robot description, xacro)
@@ -5,5 +5,5 @@
 <xacro:include filename="$(find mr_robot_description)/gazebo/mr_robot.gazebo" />
 <xacro:include filename="$(find mr_robot_description)/gazebo/mr_robot_plugins.gazebo" />
-<link name="base_link">
+<link name="base_link" gravity="0 0 -9.8">
   <inertial>
     <origin rpy="0 0 0" xyz="-0.00101458512283434 -0.0007739653318165107 0.06722998744578039"/>

Commit message: fix map frame and nav file

File: mr_robot_description/urdf/mr_robot.xacro (robot description, xacro)
@@ -5,4 +5,12 @@
 <xacro:include filename="$(find mr_robot_description)/gazebo/mr_robot.gazebo" />
 <xacro:include filename="$(find mr_robot_description)/gazebo/mr_robot_plugins.gazebo" />
+<!-- <link name ="world"> -->
+<!-- </link> -->
+<!--  -->
+<!-- <joint name="base_joint"> -->
+<!-- <type: "floating"/> -->
+<!-- <parent_frame_id: "world"/> -->
+<!-- <child_frame_id: "base_link"/> -->
+<!-- </joint> -->
 <link name="base_link" gravity="0 0 -9.8">
   <inertial>

Commit message: added ros2 launch params for plugins

File: mr_robot_description/urdf/mr_robot.xacro (robot description, xacro)
@@ -5,12 +5,7 @@
 <xacro:include filename="$(find mr_robot_description)/gazebo/mr_robot.gazebo" />
 <xacro:include filename="$(find mr_robot_description)/gazebo/mr_robot_plugins.gazebo" />
-<!-- <link name ="world"> -->
-<!-- </link> -->
-<!--  -->
-<!-- <joint name="base_joint"> -->
-<!-- <type: "floating"/> -->
-<!-- <parent_frame_id: "world"/> -->
-<!-- <child_frame_id: "base_link"/> -->
-<!-- </joint> -->
+<xacro:arg      name="kinect_enabled"             default="true" />
+<xacro:arg      name="lidar_enabled"              default="true" />
+<xacro:arg      name="camera_enabled"             default="true" />
 <link name="base_link" gravity="0 0 -9.8">
   <inertial>
@@ -73,4 +68,5 @@
   </collision>
 </link>
+<xacro:if value="$(arg lidar_enabled)">
 <link name="lidar_1">
   <inertial>
@@ -93,4 +89,63 @@
   </collision>
 </link>
+<joint name="lidar_fixed" type="fixed">
+  <origin rpy="0 0 0" xyz="0.0967 -0.001759 0.108682"/>
+  <parent link="base_link"/>
+  <child link="lidar_1"/>
+</joint>
+</xacro:if>
+<xacro:if value="$(arg kinect_enabled)">
+	<link name="kinect_camera">
+		<collision>
+		  <origin xyz="0 0 0" rpy="0 0 0" />
+		<geometry>
+			<box size="0.07 0.3 0.09"/>
+		</geometry>
+		</collision>
+		<visual>
+			<origin xyz="0 0 0" rpy="0 0 0" />
+		<geometry>
+		<mesh filename="file://$(find mr_robot_description)/meshes/kinect/d415.dae"/>
+		</geometry>
+		<material name="black"/>
+		</visual>
+		<inertial>
+			<mass value="0.01"/>
+      <inertia ixx="${0.01 / 12.0 * (0.09*0.09 + 0.3*0.3)}" ixy="0.0" ixz="0.0" iyy="${0.01 / 12.0 * (0.07*0.07 + 0.3*0.3)}" iyz="0.0" izz="${0.01 / 12.0 * (0.07*0.07 + 0.3*0.3)}"/>
+		</inertial>
+	</link>
+	<joint name="kinect_camera_joint" type="fixed">
+			<origin rpy="0 0 0" xyz="0.15 -0.001759 0.073682"/>
+			<parent link="base_link"/>
+			<child link="kinect_camera"/>
+	</joint>
+</xacro:if>
+<xacro:if value="$(arg camera_enabled)">
+  <link name="camera_link">
+    <collision>
+      <origin xyz="0 0 0" rpy="0 0 0"/>
+      <geometry>
+    <box size="0.05 0.05 0.05"/>
+        </geometry>
+    </collision>
+    <visual>
+      <origin xyz="0 0 0" rpy="0 0 0"/>
+      <geometry>
+    <box size="0.05 0.05 0.05"/>
+      </geometry>
+      <material name="red"/>
+    </visual>
+    <inertial>
+      <mass value="1e-5" />
+      <origin xyz="0 0 0" rpy="0 0 0"/>
+      <inertia ixx="1e-6" ixy="0" ixz="0" iyy="1e-6" iyz="0" izz="1e-6" />
+    </inertial>
+  </link>
+  <joint name="camera_joint" type="fixed">
+   <origin rpy="0 0 0" xyz="0.0967 -0.001759 0.163682"/>
+   <parent link="base_link"/>
+   <child link="camera_link"/>
+  </joint>
+</xacro:if>
 <joint name="right_motor_joint" type="continuous">
   <origin rpy="0 0 0" xyz="-0.003445 -0.10058 0.052283"/>
@@ -105,8 +160,3 @@
   <axis xyz="0.0 1.0 0.0"/>
 </joint>
-<joint name="lidar_fixed" type="fixed">
-  <origin rpy="0 0 0" xyz="0.0967 -0.001759 0.108682"/>
-  <parent link="base_link"/>
-  <child link="lidar_1"/>
-</joint>
 </robot>

Commit message: added ros launch params for plugins

File: mr_robot_description/urdf/mr_robot.xacro (robot description, xacro)
@@ -5,4 +5,7 @@
 <xacro:include filename="$(find mr_robot_description)/gazebo/mr_robot.gazebo" />
 <xacro:include filename="$(find mr_robot_description)/gazebo/mr_robot_plugins.gazebo" />
+<xacro:arg      name="kinect_enabled"             default="true" />
+<xacro:arg      name="lidar_enabled"              default="true" />
+<xacro:arg      name="camera_enabled"             default="true" />
 <link name="base_link">
   <inertial>
@@ -65,4 +68,5 @@
   </collision>
 </link>
+<xacro:if value="$(arg lidar_enabled)">
 <link name="lidar_1">
   <inertial>
@@ -85,4 +89,63 @@
   </collision>
 </link>
+  <joint name="lidar_fixed" type="fixed">
+  <origin rpy="0 0 0" xyz="0.0967 -0.001759 0.108682"/>
+  <parent link="base_link"/>
+  <child link="lidar_1"/>
+</joint>
+</xacro:if>
+<xacro:if value="$(arg camera_enabled)">
+ <link name="camera_link">
+    <collision>
+      <origin xyz="0 0 0" rpy="0 0 0"/>
+      <geometry>
+    <box size="0.05 0.05 0.05"/>
+        </geometry>
+    </collision>
+    <visual>
+      <origin xyz="0 0 0" rpy="0 0 0"/>
+      <geometry>
+    <box size="0.05 0.05 0.05"/>
+      </geometry>
+      <material name="red"/>
+    </visual>
+    <inertial>
+      <mass value="1e-5" />
+      <origin xyz="0 0 0" rpy="0 0 0"/>
+      <inertia ixx="1e-6" ixy="0" ixz="0" iyy="1e-6" iyz="0" izz="1e-6" />
+    </inertial>
+  </link>
+  <joint name="camera_joint" type="fixed">
+  <origin rpy="0 0 0" xyz="0.0967 -0.001759 0.163682"/>
+  <parent link="base_link"/>
+  <child link="camera_link"/>
+</joint>
+</xacro:if>
+<xacro:if value="$(arg kinect_enabled)">
+	<link name="kinect_camera">
+		<collision>
+		  <origin xyz="0 0 0" rpy="0 0 0" />
+		<geometry>
+			<box size="0.07 0.3 0.09"/>
+		</geometry>
+		</collision>
+		<visual>
+			<origin xyz="0 0 0" rpy="0 0 0" />
+		<geometry>
+		<mesh filename="file://$(find mr_robot_description)/meshes/kinect/d415.dae"/>
+		</geometry>
+		<material name="black"/>
+		</visual>
+		<inertial>
+			<mass value="0.01"/>
+      <inertia ixx="${0.01 / 12.0 * (0.09*0.09 + 0.3*0.3)}" ixy="0.0" ixz="0.0" iyy="${0.01 / 12.0 * (0.07*0.07 + 0.3*0.3)}" iyz="0.0" izz="${0.01 / 12.0 * (0.07*0.07 + 0.3*0.3)}"/>
+		</inertial>
+	</link>
+	<joint name="kinect_camera_joint" type="fixed">
+			<origin rpy="0 0 0" xyz="0.15 -0.001759 0.073682"/>
+			<parent link="base_link"/>
+			<child link="kinect_camera"/>
+	</joint>
+</xacro:if>
 <joint name="right_motor_joint" type="continuous">
   <origin rpy="0 0 0" xyz="-0.003445 -0.10058 0.052283"/>
@@ -97,8 +160,3 @@
   <axis xyz="0.0 1.0 0.0"/>
 </joint>
-<joint name="lidar_fixed" type="fixed">
-  <origin rpy="0 0 0" xyz="0.0967 -0.001759 0.108682"/>
-  <parent link="base_link"/>
-  <child link="lidar_1"/>
-</joint>
 </robot>
